Commit message: .

File: my_2wd_robot/urdf/controllers/diff_drive.urdf.xacro (robot description, xacro)
@@ -6,5 +6,5 @@
           <remapping>odom:=odom/unfiltered</remapping>
         </ros>
-        <updateRate>100</updateRate>
+        <updateRate>50</updateRate>
         <left_joint>left_wheel_joint</left_joint>
         <right_joint>right_wheel_joint</right_joint>

File: my_2wd_robot/urdf/robot_parts/base.urdf.xacro (robot description, xacro)
@@ -2,5 +2,5 @@
 <robot xmlns:xacro="http://ros.org/wiki/xacro">
   <xacro:macro name="base" params="length width height mass wheel_radius wheel_pos_z">
-    <!-- <link name="base_footprint"/> -->
+    <link name="base_footprint"/>
     <link name="base_link">
       <visual>
@@ -38,9 +38,9 @@
       </visual>
     </gazebo>
-    <!-- <joint name="base_to_footprint" type="fixed">
+    <joint name="base_to_footprint" type="fixed">
       <parent link="base_footprint"/>
       <child link="base_link"/>
       <origin xyz="0 0 ${wheel_radius - wheel_pos_z}" rpy="0 0 0"/>
-    </joint> -->
+    </joint>
   </xacro:macro>
 </robot>

File: my_2wd_robot/urdf/sensors/lidar.xacro (robot description, xacro)
@@ -43,6 +43,5 @@
             <pose> 0 0 0 0 0 0 </pose>
             <visualize>true</visualize>
-            <updateRate>10</updateRate>
-            <!-- <update_rate>10.0</update_rate> -->
+            <update_rate>50</update_rate>
             <ray>
                 <scan>
@@ -62,7 +61,8 @@
             <plugin name="laser_controller" filename="libgazebo_ros_ray_sensor.so">
                 <ros>
-                    <argument>--ros-args --remap /laser_controller/out:=/scan</argument>
+                    <remapping>laser_controller/out:=scan</remapping>
                 </ros>
                 <output_type>sensor_msgs/LaserScan</output_type>
+                <!-- <frame_name>laser_frame</frame_name> -->
             </plugin>
         </sensor>

Commit message: nav2/slam_toolbox done

File: my_2wd_robot/urdf/controllers/diff_drive.urdf.xacro (robot description, xacro)
@@ -3,7 +3,7 @@
     <gazebo>
       <plugin name="differential_drive_controller" filename="libgazebo_ros_diff_drive.so">
-        <ros>
+        <!-- <ros>
           <remapping>odom:=odom/unfiltered</remapping>
-        </ros>
+        </ros> -->
         <updateRate>50</updateRate>
         <left_joint>left_wheel_joint</left_joint>
@@ -12,7 +12,7 @@
         <wheel_diameter>${wheel_radius * 2}</wheel_diameter>
         <max_wheel_acceleration>1.0</max_wheel_acceleration>
-        <robot_base_frame>base_footprint</robot_base_frame>
+        <robot_base_frame>base_link</robot_base_frame>
         <publish_odom>true</publish_odom>
-        <publish_odom_tf>false</publish_odom_tf>
+        <publish_odom_tf>true</publish_odom_tf>
         <publish_wheel_tf>true</publish_wheel_tf>
         <odometry_frame>odom</odometry_frame>

File: my_2wd_robot/urdf/robot_parts/base.urdf.xacro (robot description, xacro)
@@ -2,5 +2,4 @@
 <robot xmlns:xacro="http://ros.org/wiki/xacro">
   <xacro:macro name="base" params="length width height mass wheel_radius wheel_pos_z">
-    <link name="base_footprint"/>
     <link name="base_link">
       <visual>
@@ -38,7 +37,9 @@
       </visual>
     </gazebo>
+    <link name="base_footprint">
+    </link>
     <joint name="base_to_footprint" type="fixed">
-      <parent link="base_footprint"/>
-      <child link="base_link"/>
+      <parent link="base_link"/>
+      <child link="base_footprint"/>
       <origin xyz="0 0 ${wheel_radius - wheel_pos_z}" rpy="0 0 0"/>
     </joint>
